File: KP1800/_autosave-KP1800.kicad_pcb (KiCad board)
At the start: 2 copper layers, 141 parts, among them J1 USB_C_Receptacle_USB2.0_14P, SW1 SW_Push, SW2 SW_Push, U1 USBLC6-2SC6, U2 STM32F072CBTx, U3 XC6206PxxxMR

Commit message: Working on PCB // Laid out key switches // 60% board
Parts:
- moved S61 205.6 mm to (247.3, 258.0)
- moved S43 191.5 mm to (247.2, 60.3)
- moved S62 190.5 mm to (342.6, 92.1)
- moved S40 180.0 mm to (190.0, 60.3)
- moved S41 166.9 mm to (209.1, 60.3)
- moved S64 166.6 mm to (275.7, 234.2)
- moved S63 161.8 mm to (251.9, 234.2)
- moved S58 161.1 mm to (49.5, 98.4)
- moved S44 160.1 mm to (278.1, 60.3)
- moved S42 154.5 mm to (228.1, 60.3)
- moved S56 148.8 mm to (273.4, 79.4)
- moved D19 132.9 mm to (336.5, 174.0)
- moved D20 132.9 mm to (336.5, 177.4)
- moved D24 132.9 mm to (336.5, 190.8)
- moved D25 132.9 mm to (336.5, 194.1)
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