File: KP1800/_autosave-KP1800.kicad_pcb (KiCad board)
At the start: 2 copper layers, 285.8 x 95.2 mm, 142 parts, among them J1 USB_C_Receptacle_USB2.0_14P, SW1 SW_Push, SW2 SW_Push, U1 USBLC6-2SC6, U2 STM32F072CBTx, U3 XC6206PxxxMR

Commit message: Added traces to matrix
Parts:
- moved U2 88.1 mm to (95.5, 114.4), turned to 90 degrees
- moved C8 20.2 mm to (68.2, 100.2)
- moved C7 16.5 mm to (67.9, 94.5)
- moved U3 11.7 mm to (95.0, 93.9), turned to -90 degrees
- moved U1 1.90 mm to (85.3, 85.2), turned to -90 degrees
- moved J1 0.86 mm to (85.3, 75.9)
- moved D1 0.32 mm to (79.4, 88.5)
Routing:
- net A4: track 0.00 -> 264.3 mm, vias 0 -> 2
- net A0: track 0.00 -> 258.6 mm, vias 0 -> 2
- net A1: track 0.00 -> 257.2 mm
- net A2: track 0.00 -> 247.7 mm
- net A3: track 0.00 -> 238.2 mm
- net B7: track 0.00 -> 187.2 mm
- net B6: track 0.00 -> 182.2 mm
- net B5: track 0.00 -> 176.8 mm
- net B4: track 0.00 -> 171.8 mm
- net B3: track 0.00 -> 119.3 mm
- net B11: track 0.00 -> 79.3 mm
- net B1: track 0.00 -> 70.3 mm
- net B2: track 0.00 -> 68.0 mm
- net B8: track 0.00 -> 67.0 mm
- net B10: track 0.00 -> 67.0 mm
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Other:
- board outline removed

Commit message: Added mounting moles + stabilizers WIP
Parts:
- added REF**: MountingHole_2.2mm_M2, MountingHole:MountingHole_2.2mm_M2, F.Cu at (326.6, 101.8)
- added REF**: MountingHole_2.2mm_M2, MountingHole:MountingHole_2.2mm_M2, F.Cu at (91.8, 101.7)
- added REF**: MountingHole_2.2mm_M2, MountingHole:MountingHole_2.2mm_M2, F.Cu at (351.6, 130.3)
- added REF**: MountingHole_2.2mm_M2, MountingHole:MountingHole_2.2mm_M2, F.Cu at (194.8, 120.8)
- added REF**: Stabilizer_MX_2.00u, ScottoKeebs_Stabilizer:Stabilizer_MX_2.00u, F.Cu at (332.9, 83.1)
- added REF**: MountingHole_2.2mm_M2, MountingHole:MountingHole_2.2mm_M2, F.Cu at (257.1, 159.1)
- added REF**: Stabilizer_MX_2.00u, ScottoKeebs_Stabilizer:Stabilizer_MX_2.00u, F.Cu at (330.5, 121.2)
- added REF**: Stabilizer_MX_2.00u, ScottoKeebs_Stabilizer:Stabilizer_MX_2.00u, F.Cu at (87.6, 140.2)
- added REF**: Stabilizer_MX_2.00u, ScottoKeebs_Stabilizer:Stabilizer_MX_2.00u, F.Cu at (325.8, 140.4)
- added REF**: MountingHole_2.2mm_M2, MountingHole:MountingHole_2.2mm_M2, F.Cu at (66.6, 130.3)
- moved REF** 0.52 mm to (197.3, 157.9)
- moved J1 0.09 mm to (85.3, 76.0)
- turned U1 to 90 degrees
Routing:
- net D-: track 4.45 -> 0.00 mm
- net D+: track 4.45 -> 0.00 mm
Other:
- board outline added: 285 x 94.6 mm
