File: KP1800/_autosave-KP1800.kicad_pcb (KiCad board)
At the start: 2 copper layers, 285 x 94.6 mm, 151 parts, among them J1 USB_C_Receptacle_USB2.0_14P, SW2 SW_Push, U1 USBLC6-2SC6, U2 STM32F072CBTx, U3 XC6206PxxxMR

Commit message: Optimized Traces + Fixed Silkscreen DRC Errors
Parts:
- moved R1 1.24 mm to (178.9, 162.2)
- renumbered REF** to H1, REF** to H2, REF** to H3, REF** to H4, REF** to H5, REF** to H6, REF** to ST1, REF** to ST2, REF** to ST3, REF** to ST4, REF** to ST5
Routing:
- net +3.3V: track 56.2 -> 214.3 mm, vias 0 -> 2
- net B31: track 309.1 -> 299.1 mm
- net A6: track 383.4 -> 374.5 mm
- net B30: track 334.9 -> 327.2 mm
- net +5V: track 11.5 -> 18.5 mm, vias 0 -> 2
- net A5: track 406.1 -> 400.9 mm, vias 9 -> 8
- net A4: track 434.2 -> 430.9 mm
- net B9: track 337.6 -> 334.5 mm
- net A3: track 449.0 -> 446.2 mm
- net A8: track 296.3 -> 294.0 mm
- net GND: track 40.2 -> 41.5 mm

Commit message: Added Ground Filled Zones + Finished All Traces  // Working on final touches
Routing:
- net GND: track 41.5 -> 64.7 mm, vias 0 -> 6
- net VBUS: track 5.79 -> 13.2 mm, vias 0 -> 2
- net +3.3V: track 214.3 -> 218.0 mm, vias 2 -> 4
- net B8: track 191.3 -> 189.4 mm
- added copper zone on B.Cu, net GND
- added copper zone on F.Cu, net GND
