File: KP1800/KP1800.kicad_pcb (KiCad board)
At the start: 2 copper layers, 141 parts, among them J1 USB_C_Receptacle_USB2.0_14P, SW1 SW_Push, SW2 SW_Push, U1 USBLC6-2SC6, U2 STM32F072CBTx, U3 XC6206PxxxMR

Commit message: Cleaned up rats nest
Parts:
- added REF**: Stabilizer_MX_6.25u, ScottoKeebs_Stabilizer:Stabilizer_MX_6.25u, F.Cu at (144.9, 97.6)
- moved D1 252.8 mm to (28.6, 26.2), turned to 90 degrees
- moved D15 242.1 mm to (33.3, 45.2), turned to 90 degrees
- moved D2 234.5 mm to (47.6, 26.2), turned to 90 degrees
- moved D29 226.0 mm to (35.7, 64.3), turned to 90 degrees
- moved D54 219.7 mm to (31.0, 102.4), turned to 90 degrees
- moved D16 219.0 mm to (57.1, 45.2), turned to 90 degrees
- moved D3 216.3 mm to (66.7, 26.2), turned to 90 degrees
- moved D42 215.5 mm to (40.5, 83.3), turned to 90 degrees
- moved D17 200.8 mm to (76.2, 45.3), turned to 90 degrees
- moved D30 199.8 mm to (61.9, 64.3), turned to 90 degrees
- moved D4 198.4 mm to (85.7, 26.2), turned to 90 degrees
- moved D55 194.1 mm to (54.8, 102.4), turned to 90 degrees
- moved S43 191.5 mm to (247.2, 60.3)
- moved D43 184.5 mm to (71.4, 83.3), turned to 90 degrees
- moved D18 182.9 mm to (95.2, 45.2), turned to 90 degrees
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