File: KP1800/KP1800.kicad_pcb (KiCad board)
At the start: 2 copper layers, 285.8 x 95.2 mm, 142 parts, among them J1 USB_C_Receptacle_USB2.0_14P, SW1 SW_Push, SW2 SW_Push, U1 USBLC6-2SC6, U2 STM32F072CBTx, U3 XC6206PxxxMR

Commit message: Added mounting moles + stabilizers WIP
Parts:
- added REF**: Standoff_M2x6mm, ScottoKeebs_Scotto:Standoff_M2x6mm, F.Cu at (91.8, 101.7)
- moved U2 88.1 mm to (95.5, 114.4), turned to 90 degrees
- moved C8 20.2 mm to (68.2, 100.2)
- moved C7 16.5 mm to (67.9, 94.5)
- moved U3 11.7 mm to (95.0, 93.9), turned to -90 degrees
- moved U1 1.90 mm to (85.3, 85.2)
- moved J1 0.86 mm to (85.3, 76.0)
- moved D1 0.32 mm to (79.4, 88.5)
Routing:
- net A4: track 0.00 -> 264.3 mm, vias 0 -> 2
- net A0: track 0.00 -> 258.6 mm, vias 0 -> 2
- net A1: track 0.00 -> 257.2 mm
- net A2: track 0.00 -> 247.7 mm
- net A3: track 0.00 -> 238.2 mm
- net B7: track 0.00 -> 187.2 mm
- net B6: track 0.00 -> 182.2 mm
- net B5: track 0.00 -> 176.8 mm
- net B4: track 0.00 -> 171.8 mm
- net B3: track 0.00 -> 119.3 mm
- net B11: track 0.00 -> 79.3 mm
- net B1: track 0.00 -> 70.3 mm
- net B2: track 0.00 -> 68.0 mm
- net B8: track 0.00 -> 67.0 mm
- net B10: track 0.00 -> 67.0 mm
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Other:
- board size 285.8 x 95.2 mm -> 285 x 94.6 mm

Commit message: 80% of signal traces are complete
Parts:
- removed the REF** at (91.8, 101.7)
- added REF**: MountingHole_2.2mm_M2, MountingHole:MountingHole_2.2mm_M2, F.Cu at (326.6, 101.8)
- added REF**: MountingHole_2.2mm_M2, MountingHole:MountingHole_2.2mm_M2, F.Cu at (91.8, 101.7)
- added REF**: MountingHole_2.2mm_M2, MountingHole:MountingHole_2.2mm_M2, F.Cu at (351.6, 130.3)
- added REF**: MountingHole_2.2mm_M2, MountingHole:MountingHole_2.2mm_M2, F.Cu at (194.8, 120.8)
- added REF**: Stabilizer_MX_2.00u, ScottoKeebs_Stabilizer:Stabilizer_MX_2.00u, F.Cu at (332.9, 83.1)
- added REF**: MountingHole_2.2mm_M2, MountingHole:MountingHole_2.2mm_M2, F.Cu at (257.1, 159.1)
- added REF**: Stabilizer_MX_2.00u, ScottoKeebs_Stabilizer:Stabilizer_MX_2.00u, F.Cu at (330.5, 121.2)
- added REF**: Stabilizer_MX_2.00u, ScottoKeebs_Stabilizer:Stabilizer_MX_2.00u, F.Cu at (87.6, 140.2)
- added REF**: Stabilizer_MX_2.00u, ScottoKeebs_Stabilizer:Stabilizer_MX_2.00u, F.Cu at (325.8, 140.4)
- added REF**: MountingHole_2.2mm_M2, MountingHole:MountingHole_2.2mm_M2, F.Cu at (66.6, 130.3)
- moved U2 87.9 mm to (170.9, 159.6)
- moved C7 27.2 mm to (95.1, 94.5), turned to 90 degrees
- moved F1 18.1 mm to (89.0, 86.8)
- moved C5 17.2 mm to (160.7, 156.8), turned to -90 degrees
- moved C4 14.7 mm to (180.1, 162.2), turned to 90 degrees
- moved C9 9.65 mm to (161.7, 152.5)
- moved C6 5.92 mm to (177.6, 162.3), turned to 90 degrees
- moved SW1 5.52 mm to (155.1, 155.9)
- moved U3 4.05 mm to (91.0, 93.9)
- moved SW2 2.13 mm to (186.0, 162.2)
- moved C1 1.46 mm to (169.9, 166.0)
- moved C2 1.37 mm to (163.5, 156.8)
- moved R3 1.00 mm to (79.0, 79.5)
- moved C3 0.90 mm to (174.4, 152.9)
- moved REF** 0.52 mm to (197.3, 157.9)
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Connections:
- D1 pad 1: A0 -> A3
- D10 pad 1: A0 -> A3
- D11 pad 1: A0 -> A3
- D12 pad 1: A0 -> A3
- D13 pad 1: A0 -> A3
- D14 pad 1: A0 -> A3
- D15 pad 1: A1 -> A4
- D16 pad 1: A1 -> A4
- D17 pad 1: A1 -> A4
- D18 pad 1: A1 -> A4
- D19 pad 1: A1 -> A4
- D2 pad 1: A0 -> A3
- D20 pad 1: A1 -> A4
- D21 pad 1: A1 -> A4
- D22 pad 1: A1 -> A4
- D23 pad 1: A1 -> A4
- D24 pad 1: A1 -> A4
- D25 pad 1: A1 -> A4
- D26 pad 1: A1 -> A4
- D27 pad 1: A1 -> A4
- D28 pad 1: A1 -> A4
- D29 pad 1: A2 -> A5
- D3 pad 1: A0 -> A3
- D30 pad 1: A2 -> A5
- D31 pad 1: A2 -> A5
- D32 pad 1: A2 -> A5
- D33 pad 1: A2 -> A5
- D34 pad 1: A2 -> A5
- D35 pad 1: A2 -> A5
- D36 pad 1: A2 -> A5
- D37 pad 1: A2 -> A5
- D38 pad 1: A2 -> A5
- D39 pad 1: A2 -> A5
- D4 pad 1: A0 -> A3
- D40 pad 1: A2 -> A5
- D41 pad 1: A2 -> A5
- D42 pad 1: A3 -> A6
- D43 pad 1: A3 -> A6
- D44 pad 1: A3 -> A6
- D45 pad 1: A3 -> A6
- D46 pad 1: A3 -> A6
- D47 pad 1: A3 -> A6
- D48 pad 1: A3 -> A6
- D49 pad 1: A3 -> A6
- D5 pad 1: A0 -> A3
- D50 pad 1: A3 -> A6
- D51 pad 1: A3 -> A6
- D52 pad 1: A3 -> A6
- D53 pad 1: A3 -> A6
- D54 pad 1: A4 -> A7
- D55 pad 1: A4 -> A7
- D56 pad 1: A4 -> A7
- D57 pad 1: A4 -> A7
- D58 pad 1: A4 -> A7
- D59 pad 1: A4 -> A7
- D6 pad 1: A0 -> A3
- D60 pad 1: A4 -> A7
- D61 pad 1: A4 -> A7
- D7 pad 1: A0 -> A3
- D8 pad 1: A0 -> A3
- D9 pad 1: A0 -> A3
- S1 pad 1: B0 -> B12
- S10 pad 1: B9 -> B8
- S11 pad 1: B10 -> B9
- S12 pad 1: B11 -> B30
- S13 pad 1: B12 -> B31
- S14 pad 1: B13 -> A8
- S18 pad 1: B0 -> B12
- S19 pad 1: B1 -> B13
- S2 pad 1: B1 -> B13
- S20 pad 1: B2 -> B14
- S21 pad 1: B3 -> B15
- S22 pad 1: B4 -> B3
- S23 pad 1: B5 -> B4
- S24 pad 1: B6 -> B5
- S25 pad 1: B7 -> B6
- S26 pad 1: B8 -> B7
- S27 pad 1: B9 -> B8
- S28 pad 1: B10 -> B9
- S29 pad 1: B11 -> B30
- S3 pad 1: B2 -> B14
- S30 pad 1: B12 -> B31
- S31 pad 1: B13 -> A8
- S32 pad 1: B0 -> B12
- S33 pad 1: B1 -> B13
- S34 pad 1: B2 -> B14
- S35 pad 1: B3 -> B15
- S36 pad 1: B4 -> B3
- S37 pad 1: B5 -> B4
- S38 pad 1: B6 -> B5
- S39 pad 1: B7 -> B6
- S4 pad 1: B3 -> B15
- S40 pad 1: B8 -> B7
- S41 pad 1: B9 -> B8
- S42 pad 1: B10 -> B9
- S43 pad 1: B11 -> B30
- S44 pad 1: B12 -> B31
- S45 pad 1: B0 -> B12
- S46 pad 1: B1 -> B13
- S47 pad 1: B2 -> B14
- S48 pad 1: B3 -> B15
- S49 pad 1: B4 -> B3
- S5 pad 1: B4 -> B3
- S50 pad 1: B5 -> B4
- S51 pad 1: B6 -> B5
- S52 pad 1: B7 -> B6
- S53 pad 1: B8 -> B7
- S54 pad 1: B9 -> B8
- S55 pad 1: B10 -> B9
- S56 pad 1: B11 -> B30
- S57 pad 1: B0 -> B12
- S58 pad 1: B1 -> B13
- S59 pad 1: B2 -> B14
- S6 pad 1: B5 -> B4
- S60 pad 1: B3 -> B15
- S61 pad 1: B4 -> B3
- S62 pad 1: B5 -> B4
- S63 pad 1: B6 -> B5
- S64 pad 1: B7 -> B6
- S7 pad 1: B6 -> B5
- S8 pad 1: B7 -> B6
- S9 pad 1: B8 -> B7
- U2 pad 10: A0 -> unconnected-(U2-PA0-Pad10)
- U2 pad 11: A1 -> unconnected-(U2-PA1-Pad11)
- U2 pad 12: A2 -> unconnected-(U2-PA2-Pad12)
- U2 pad 15: unconnected-(U2-PA5-Pad15) -> A5
- U2 pad 16: unconnected-(U2-PA6-Pad16) -> A6
- U2 pad 17: unconnected-(U2-PA7-Pad17) -> A7
- U2 pad 18: B0 -> unconnected-(U2-PB0-Pad18)
- U2 pad 19: B1 -> unconnected-(U2-PB1-Pad19)
- U2 pad 20: B2 -> unconnected-(U2-PB2-Pad20)
- U2 pad 21: B10 -> unconnected-(U2-PB10-Pad21)
- U2 pad 22: B11 -> unconnected-(U2-PB11-Pad22)
- U2 pad 27: unconnected-(U2-PB14-Pad27) -> B14
- U2 pad 28: unconnected-(U2-PB15-Pad28) -> B15
- U2 pad 29: unconnected-(U2-PA8-Pad29) -> A8
- U2 pad 30: unconnected-(U2-PA9-Pad30) -> B30
- U2 pad 31: unconnected-(U2-PA10-Pad31) -> B31
Routing:
- net A5: track 0.00 -> 406.1 mm, vias 0 -> 9
- net A6: track 0.00 -> 383.4 mm, vias 0 -> 8
- net A7: track 0.00 -> 362.1 mm, vias 0 -> 4
- net B30: track 0.00 -> 334.9 mm, vias 0 -> 1
- net B31: track 0.00 -> 309.1 mm, vias 0 -> 1
- net A8: track 0.00 -> 296.3 mm, vias 0 -> 1
- net B9: track 67.0 -> 337.6 mm, vias 0 -> 1
- net A0: track 258.6 -> 0.00 mm, vias 2 -> 0
- net A1: track 257.2 -> 0.00 mm
- net A2: track 247.7 -> 0.00 mm
- net A3: track 238.2 -> 449.0 mm, vias 0 -> 2
- net D+: track 0.00 -> 180.8 mm
- net D-: track 0.00 -> 180.8 mm, vias 0 -> 2
- net A4: track 264.3 -> 434.2 mm
- net B15: track 0.00 -> 129.5 mm, vias 0 -> 1
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
Commit message: Added Ground Filled Zones + Finished All Traces  // Working on final touches
Parts:
- removed SW1: SW_Push, Button_Switch_SMD:SW_SPST_TL3342
- moved C8 26.9 mm to (93.3, 90.7), turned to 0 degrees
- moved C9 17.5 mm to (172.5, 166.3), turned to 180 degrees
- moved R1 5.06 mm to (178.9, 162.2), turned to -90 degrees
- moved C6 4.95 mm to (176.7, 167.1), turned to 180 degrees
- moved C4 4.42 mm to (176.7, 165.0), turned to 180 degrees
- moved SW2 2.00 mm to (184.2, 163.2), turned to 0 degrees
- moved C1 1.50 mm to (168.4, 166.3)
- moved C7 0.79 mm to (94.5, 93.9)
- renumbered REF** to H1, REF** to H2, REF** to H3, REF** to H4, REF** to H5, REF** to H6, REF** to ST1, REF** to ST2, REF** to ST3, REF** to ST4, REF** to ST5
Routing:
- net +3.3V: track 5.46 -> 214.3 mm, vias 0 -> 2
- net B12: track 79.5 -> 180.8 mm
- net B13: track 85.0 -> 164.8 mm, vias 0 -> 2
- net B14: track 92.2 -> 149.3 mm, vias 0 -> 2
- net +5V: track 5.75 -> 18.5 mm, vias 0 -> 2
- net BOOT0: track 0.00 -> 12.7 mm
- net GND: track 29.5 -> 41.5 mm
- net B31: track 309.1 -> 299.1 mm
- net A6: track 383.4 -> 374.5 mm
- net B30: track 334.9 -> 327.2 mm
- net A5: track 406.1 -> 400.9 mm, vias 9 -> 8
- net A4: track 434.2 -> 430.9 mm
- net B9: track 337.6 -> 334.5 mm
- net /NRST: track 0.00 -> 2.85 mm
- net A3: track 449.0 -> 446.2 mm
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
Commit message: Adding silkscreen + polish
Parts:
- moved H1 0.16 mm to (351.4, 130.3)
- moved H2 0.15 mm to (66.7, 130.3)
Routing:
- net GND: track 41.5 -> 64.7 mm, vias 0 -> 6
- net VBUS: track 5.79 -> 13.2 mm, vias 0 -> 2
- net +3.3V: track 214.3 -> 218.0 mm, vias 2 -> 4
- net B8: track 191.3 -> 189.4 mm
- added copper zone on B.Cu, net GND
- added copper zone on F.Cu, net GND

Commit message: Polishing Cont.
Parts:
- added G***: LOGO, LOGO, F.Cu at (222.3, 158.1)
Routing:
- net GND: track 64.7 -> 61.9 mm
- net A3: track 446.2 -> 447.4 mm
