File: KP60/matrix.kicad_sch (KiCad schematic)
At the start: 122 parts

Commit message: more images + naming fixes
Other:
- title: KP1800 Matrix -> KP60 Matrix
Changed lines of the file:
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@@
 	(paper "A4")
 	(title_block
-		(title "KP1800 Matrix")
-		(date "2025-05-02")
+		(title "KP60 Matrix")
+		(date "2025-05-03")
 		(rev "0.1")
 	)

Commit message: polish
Other:
- note added: "Diode Matrix"
- moved on the sheet: D1, D10, D11, D12, D13, D15, D16, D17, D18, D19, D2, D20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
