File: KP60/_autosave-KP60.kicad_sch (KiCad schematic)
At the start: 18 parts, among them J1 USB_C_Receptacle_USB2.0_14P, SW2 SW_Push, U1 USBLC6-2SC6, U2 STM32F072CBTx, U3 XC6206PxxxMR

Commit message: add led matrix circuit + passed ERC
Connections:
- net A2: now reaches U2.12 (PA2)
- no-connect marks 16 -> 15
Other:
- added sheet RGB (RGB_sch.kicad_sch)
Changed lines of the file:
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@@
 	)
 	(no_connect
-		(at 116.84 64.77)
-	)
-	(no_connect
 		(at 83.82 77.47)
 	)
@@
 		)
 	)
+	(global_label "A2"
+		(shape input)
+		(at 116.84 64.77 0)
+		(fields_autoplaced yes)
+		(effects
+			(font
+				(size 1.27 1.27)
+			)
+			(justify left)
+		)
+		(property "Intersheetrefs" "${INTERSHEET_REFS}"
+			(at 122.1233 64.77 0)
+			(effects
+				(font
+					(size 1.27 1.27)
+				)
+				(justify left)
+				(hide yes)
+			)
+		)
+	)
 	(global_label "B7"
 		(shape input)
@@
 				)
 			)
+		)
+	)
+	(sheet
+		(at 10.16 441.96)
+		(size 278.13 189.23)
+		(fields_autoplaced yes)
+		(stroke
+			(width 0.1524)
+			(type solid)
+		)
+		(fill
+			(color 0 0 0 0.0000)
+		)
+		(property "Sheetname" "RGB"
+			(at 10.16 441.2484 0)
+			(effects
+				(font
+					(size 1.27 1.27)
+				)
+				(justify left bottom)
+			)
+		)
+		(property "Sheetfile" "RGB_sch.kicad_sch"
+			(at 10.16 631.7746 0)
+			(effects
+				(font
+					(size 1.27 1.27)
+				)
+				(justify left top)
+			)
+		)
+		(instances
+			(project "KP60"
+				(path "/7108c105-5751-4eb7-aac4-6c879069d1a1"
+					(page "3")
+				)
+			)
