File: KP60/RGB_sch.kicad_sch (KiCad schematic)
At the start: 88 parts

Commit message: Formatting Changes
Parts:
- added C54, C55, C56, C57, C58, C59, C60, C61, C62, C63, C64, C65, C66, C67, C68, C69, C70: 100n, symbol Device:C_Small
- added D106, D107, D108, D109, D110, D111, D112, D113, D114, D115, D116, D117, D118, D119, D120, D121, D122: LED_WS2812B, ScottoKeebs_Components:LED_WS2812B, symbol ScottoKeebs:LED_WS2812B
- C10, C11, C12, C13, C14, C15, C16, C17, C18, C19, C20, C21, C22, C23, C24, C25, C26, C27, C28, C29, C30, C31, C32, C33, C34, C35, C36, C37, C38, C39, C40, C41, C42, C43, C44, C45, C46, C47, C48, C49, C50, C51, C52, C53: value 100nF -> 100n
Connections:
- net +5V: now also D100.1 (VDD), D101.1 (VDD), D102.1 (VDD), D103.1 (VDD), D104.1 (VDD), D105.1 (VDD), D62.1 (VDD), D63.1 (VDD), D64.1 (VDD), D65.1 (VDD), D66.1 (VDD), D67.1 (VDD), D68.1 (VDD), D69.1 (VDD), D70.1 (VDD), D71.1 (VDD), D72.1 (VDD), D73.1 (VDD), D74.1 (VDD), D75.1 (VDD), D76.1 (VDD), D77.1 (VDD), D78.1 (VDD), D79.1 (VDD), D80.1 (VDD), D81.1 (VDD), D82.1 (VDD), D83.1 (VDD), D84.1 (VDD), D85.1 (VDD), D86.1 (VDD), D87.1 (VDD), D88.1 (VDD), D89.1 (VDD), D90.1 (VDD), D91.1 (VDD), D92.1 (VDD), D93.1 (VDD), D94.1 (VDD), D95.1 (VDD), D96.1 (VDD), D97.1 (VDD), D98.1 (VDD), D99.1 (VDD), C54.1, C55.1, C56.1, C57.1, C58.1, C59.1, C60.1, C61.1, C62.1, C63.1, C64.1, C65.1, C66.1, C67.1, C68.1, C69.1, C70.1, D106.1 (VDD), D107.1 (VDD), D108.1 (VDD), D109.1 (VDD), D110.1 (VDD), D111.1 (VDD), D112.1 (VDD), D113.1 (VDD), D114.1 (VDD), D115.1 (VDD), D116.1 (VDD), D117.1 (VDD), D118.1 (VDD), D119.1 (VDD), D120.1 (VDD), D121.1 (VDD), D122.1 (VDD)
- net GND: now also C10.2, C11.2, C12.2, C13.2, C14.2, C15.2, C16.2, C17.2, C18.2, C19.2, C20.2, C21.2, C22.2, C23.2, C24.2, C25.2, C26.2, C27.2, C28.2, C29.2, C30.2, C31.2, C32.2, C33.2, C34.2, C35.2, C36.2, C37.2, C38.2, C39.2, C40.2, C41.2, C42.2, C43.2, C44.2, C45.2, C46.2, C47.2, C48.2, C49.2, C50.2, C51.2, C52.2, C53.2, C54.2, C55.2, C56.2, C57.2, C58.2, C59.2, C60.2, C61.2, C62.2, C63.2, C64.2, C65.2, C66.2, C67.2, C68.2, C69.2, C70.2, D106.3 (VSS), D107.3 (VSS), D108.3 (VSS), D109.3 (VSS), D110.3 (VSS), D111.3 (VSS), D112.3 (VSS), D113.3 (VSS), D114.3 (VSS), D115.3 (VSS), D116.3 (VSS), D117.3 (VSS), D118.3 (VSS), D119.3 (VSS), D120.3 (VSS), D121.3 (VSS), D122.3 (VSS)
- net at D84.4 (DIN): now also D83.2 (DOUT)
- net at D94.2 (DOUT): now also D95.4 (DIN)
- net at D105.2 (DOUT): now also D106.4 (DIN)
- net A2: now reaches D62.4 (DIN)
- new net: D70.2 (DOUT), D71.4 (DIN)
- new net: D69.2 (DOUT), D70.4 (DIN)
- new net: D76.2 (DOUT), D77.4 (DIN)
- new net: D75.2 (DOUT), D76.4 (DIN)
- new net: D71.2 (DOUT), D72.4 (DIN)
- new net: D67.2 (DOUT), D68.4 (DIN)
- new net: D66.2 (DOUT), D67.4 (DIN)
- new net: D81.2 (DOUT), D82.4 (DIN)
- new net: D80.2 (DOUT), D81.4 (DIN)
- new net: D100.4 (DIN), D99.2 (DOUT)
- new net: D98.2 (DOUT), D99.4 (DIN)
- new net: D102.2 (DOUT), D103.4 (DIN)
- new net: D101.2 (DOUT), D102.4 (DIN)
- new net: D103.2 (DOUT), D104.4 (DIN)
- new net: D79.2 (DOUT), D80.4 (DIN)
- new net: D64.2 (DOUT), D65.4 (DIN)
- new net: D111.2 (DOUT), D112.4 (DIN)
- new net: D110.2 (DOUT), D111.4 (DIN)
- new net: D109.2 (DOUT), D110.4 (DIN)
- new net: D108.2 (DOUT), D109.4 (DIN)
- new net: D113.2 (DOUT), D114.4 (DIN)
- new net: D112.2 (DOUT), D113.4 (DIN)
- new net: D88.2 (DOUT), D89.4 (DIN)
- new net: D87.2 (DOUT), D88.4 (DIN)
- new net: D93.2 (DOUT), D94.4 (DIN)
- new net: D107.2 (DOUT), D108.4 (DIN)
- new net: D78.2 (DOUT), D79.4 (DIN)
- new net: D92.2 (DOUT), D93.4 (DIN)
- new net: D91.2 (DOUT), D92.4 (DIN)
- new net: D119.2 (DOUT), D120.4 (DIN)
- new net: D118.2 (DOUT), D119.4 (DIN)
- new net: D121.2 (DOUT), D122.4 (DIN)
- new net: D120.2 (DOUT), D121.4 (DIN)
- new net: D116.2 (DOUT), D117.4 (DIN)
- new net: D115.2 (DOUT), D116.4 (DIN)
- new net: D114.2 (DOUT), D115.4 (DIN)
- new net: D82.2 (DOUT), D83.4 (DIN)
- new net: D65.2 (DOUT), D66.4 (DIN)
- new net: D89.2 (DOUT), D90.4 (DIN)
- new net: D106.2 (DOUT), D107.4 (DIN)
- new net: D117.2 (DOUT), D118.4 (DIN)
- new net: D68.2 (DOUT), D69.4 (DIN)
- new net: D86.2 (DOUT), D87.4 (DIN)
- new net: D97.2 (DOUT), D98.4 (DIN)
- new net: D104.2 (DOUT), D105.4 (DIN)
- new net: D77.2 (DOUT), D78.4 (DIN)
- new net: D100.2 (DOUT), D101.4 (DIN)
- new net: D90.2 (DOUT), D91.4 (DIN)
- no-connect marks 0 -> 1
Other:
- note added: "LED Matrix"
- moved on the sheet: C10, D62
