File: KP60/KP60.kicad_pcb (KiCad board)
At the start: 2 copper layers, 285 x 94.6 mm, 152 parts, among them J1 USB_C_Receptacle_USB2.0_14P, SW2 SW_Push, U1 USBLC6-2SC6, U2 STM32F072CBTx, U3 XC6206PxxxMR

Commit message: Mechanical Changes
Parts:
- removed H1, H2, H3, H4, H5, H6: MountingHole_2.2mm_M2, MountingHole:MountingHole_2.2mm_M2

Commit message: Misc
Parts:
- added H1: MountingHole_2.2mm_M2, MountingHole:MountingHole_2.2mm_M2, F.Cu at (351.4, 130.3)
- added H2: MountingHole_2.2mm_M2, MountingHole:MountingHole_2.2mm_M2, F.Cu at (66.7, 130.3)
- added H3: MountingHole_2.2mm_M2, MountingHole:MountingHole_2.2mm_M2, F.Cu at (91.8, 101.8)
- added H4: MountingHole_2.2mm_M2, MountingHole:MountingHole_2.2mm_M2, F.Cu at (326.6, 101.8)
- added H5: MountingHole_2.2mm_M2, MountingHole:MountingHole_2.2mm_M2, F.Cu at (194.8, 120.8)
- added H6: MountingHole_2.2mm_M2, MountingHole:MountingHole_2.2mm_M2, F.Cu at (257.1, 159.1)
- moved J1 0.51 mm to (84.8, 76.0)

Commit message: diff. trace tweaks
Parts:
- moved R2 3.48 mm to (91.9, 76.2)
- moved R3 3.37 mm to (77.9, 76.4)
Routing:
- net Net-(J1-CC1): track 11.0 -> 7.92 mm
- net Net-(J1-CC2): track 10.8 -> 7.67 mm
- net GND: track 61.9 -> 60.4 mm
- net D-: track 183.1 -> 184.1 mm
